Commit message: nueva estructuracion

File: src/camera_description/urdf/camera.urdf.xacro (robot description, xacro)
@@ -1,69 +1,20 @@
 <?xml version="1.0"?>
-<robot name="camera" xmlns:xacro="http://www.ros.org/wiki/xacro">
-  <!-- Enlace base / soporte -->
-  <link name="camera_mount_link">
-    <visual>
-      <geometry>
-        <mesh filename="package://tu_paquete/meshes/camera_mount.stl"/>
-      </geometry>
-      <material name="gris">
-        <color rgba="0.3 0.3 0.3 1.0"/>
-      </material>
-    </visual>
-    <collision>
-      <geometry>
-        <mesh filename="package://tu_paquete/meshes/camera_mount.stl"/>
-      </geometry>
-    </collision>
-  </link>
-  <!-- Cuerpo de la cámara -->
-  <link name="camera_body_link">
-    <visual>
-      <geometry>
-        <mesh filename="package://tu_paquete/meshes/camera_body.stl"/>
-      </geometry>
-      <material name="negro">
-        <color rgba="0.05 0.05 0.05 1.0"/>
-      </material>
-    </visual>
-    <collision>
-      <geometry>
-        <mesh filename="package://tu_paquete/meshes/camera_body.stl"/>
-      </geometry>
-    </collision>
-  </link>
-  <joint name="mount_to_body" type="fixed">
-    <parent link="camera_mount_link"/>
-    <child link="camera_body_link"/>
-    <origin xyz="0 0 0.02" rpy="0 0 0"/>
-  </joint>
-  <!-- Lente -->
-  <link name="camera_lens_link">
-    <visual>
-      <geometry>
-        <mesh filename="package://tu_paquete/meshes/camera_lens.stl"/>
-      </geometry>
-      <material name="vidrio">
-        <color rgba="0.1 0.1 0.15 1.0"/>
-      </material>
-    </visual>
-    <collision>
-      <geometry>
-        <mesh filename="package://tu_paquete/meshes/camera_lens.stl"/>
-      </geometry>
-    </collision>
-  </link>
-  <joint name="body_to_lens" type="fixed">
-    <parent link="camera_body_link"/>
-    <child link="camera_lens_link"/>
-    <origin xyz="0 0 0" rpy="0 0 0"/>
-  </joint>
-  <!-- Frame óptico, útil para publicar sensor_msgs/Image o CameraInfo -->
-  <link name="camera_optical_frame"/>
-  <joint name="lens_to_optical" type="fixed">
-    <parent link="camera_lens_link"/>
-    <!-- Rotación estándar REP-103: Z hacia adelante, X derecha, Y abajo -->
-    <origin xyz="0.02 0 0" rpy="-1.5708 0 -1.5708"/>
-    <child link="camera_optical_frame"/>
-  </joint>
+<robot name="camera_robot" xmlns:xacro="http://www.ros.org/wiki/xacro">
+    <!-- Frame de proyección en el suelo -->
+    <link name="base_footprint" />
+    <!-- Link principal con tu archivo .stl -->
+    <link name="base_link">
+        <visual>
+            <geometry>
+                <mesh filename="package://camera_description/meshes/base.stl" scale="1.0 1.0 1.0"/>
+            </geometry>
+            <origin xyz="0 0 0" rpy="0 0 0" />
+        </visual>
+    </link>
+    <!-- Joint que conecta ambos para que robot_state_publisher publique el /tf -->
+    <joint name="base_joint" type="fixed">
+        <parent link="base_footprint" />
+        <child link="base_link" />
+        <origin xyz="0 0 0" rpy="0 0 0"/>
+    </joint>
 </robot>

Commit message: Ultimos cmabios

File: src/camera_description/urdf/camera.urdf.xacro (robot description, xacro)
@@ -1,20 +1,88 @@
 <?xml version="1.0"?>
 <robot name="camera_robot" xmlns:xacro="http://www.ros.org/wiki/xacro">
+    <xacro:include filename="common_properties.urdf.xacro" />
+    <xacro:arg name="package_name" default="camera_description" />
+    <xacro:arg name="mesh_dir" default="meshes" />
+    <xacro:property name="global_scale" value="1.0" />
+    <!-- Base -->
+    <xacro:property name="base_mesh" value="base.STL" />
+    <xacro:property name="base_scale" value="${global_scale} ${global_scale} ${global_scale}" />
+    <xacro:property name="base_visual_xyz" value="0 0 0" />
+    <xacro:property name="base_visual_rpy" value="0 0 0" />
+    <!-- cuerpo en u -->
+    <xacro:property name="body_u_mesh" value="cuerpo_u.STL" />
+    <xacro:property name="body_u_scale" value="${global_scale} ${global_scale} ${global_scale}" />
+    <xacro:property name="body_u_xyz" value="0 0 0.045" />
+    <xacro:property name="body_u_rpy" value="0 0 0" />
+    <xacro:property name="body_u_visual_xyz" value="0 0 0" />
+    <xacro:property name="body_u_visual_rpy" value="0 0 0" />
+    <xacro:property name="body_u_axis" value="0 0 1" />
+    <!-- cuerpo camara -->
+    <xacro:property name="camera_lens_mesh" value="lente_v3.STL" />
+    <xacro:property name="camera_lens_scale" value="${global_scale} ${global_scale*0.85} ${global_scale*0.85}" />
+    <xacro:property name="camera_lens_xyz" value="0 0.03 0.085" />
+    <xacro:property name="camera_lens_rpy" value="0 0 0" />
+    <xacro:property name="camera_lens_axis" value="1 0 0" />
+    <xacro:property name="camera_lens_visual_xyz" value="0 0 0" />
+    <xacro:property name="camera_lens_visual_rpy" value="0 0 1.5708" />
+    <!-- Macros auxiliares -->
+    <!-- Link tipo base -->
+    <xacro:macro name="mesh_link_base" params="name mesh scale">
+        <link name="${name}">
+            <visual>
+                <origin xyz="${base_visual_xyz}" rpy="${base_visual_rpy}" />
+                <geometry>
+                    <mesh filename="package://$(arg package_name)/$(arg mesh_dir)/${mesh}"
+                        scale="${scale}" />
+                </geometry>
+                <material name="white" />
+            </visual>
+        </link>
+    </xacro:macro>
+    <xacro:macro name="mesh_link_sphere" params="name mesh scale">
+        <link name="${name}">
+            <visual>
+                <origin xyz="${camera_lens_visual_xyz}" rpy="${camera_lens_visual_rpy}" />
+                <geometry>
+                    <mesh filename="package://$(arg package_name)/$(arg mesh_dir)/${mesh}"
+                        scale="${scale}" />
+                </geometry>
+                <material name="white" />
+            </visual>
+        </link>
+    </xacro:macro>
+    <!-- Instancia de Macros-links -->
     <!-- Frame de proyección en el suelo -->
     <link name="base_footprint" />
-    <!-- Link principal con tu archivo .stl -->
-    <link name="base_link">
-        <visual>
-            <geometry>
-                <mesh filename="package://camera_description/meshes/base.stl" scale="1.0 1.0 1.0"/>
-            </geometry>
-            <origin xyz="0 0 0" rpy="0 0 0" />
-        </visual>
-    </link>
-    <!-- Joint que conecta ambos para que robot_state_publisher publique el /tf -->
+    <xacro:mesh_link_base
+        name="base_link"
+        mesh="${base_mesh}"
+        scale="${base_scale}" />
+    <xacro:mesh_link_base
+        name="body_u_link"
+        mesh="${body_u_mesh}"
+        scale="${body_u_scale}" />
+    <xacro:mesh_link_sphere
+        name="camera_lens_link"
+        mesh="${camera_lens_mesh}"
+        scale="${camera_lens_scale}" />
+    <!-- Joints -->
     <joint name="base_joint" type="fixed">
         <parent link="base_footprint" />
         <child link="base_link" />
-        <origin xyz="0 0 0" rpy="0 0 0"/>
+        <origin xyz="0 0 0" rpy="0 0 0" />
+    </joint>
+    <joint name="body_u_joint" type="continuous">
+        <parent link="base_link" />
+        <child link="body_u_link" />
+        <origin xyz="0 0 0.045" rpy="0 0 0" />
+        <axis xyz="0 0 1" />
+    </joint>
+    <joint name="camera_lens_joint" type="revolute">
+        <origin xyz="${camera_lens_xyz}" rpy="${camera_lens_rpy}" />
+        <parent link="body_u_link" />
+        <child link="camera_lens_link" />
+        <axis xyz="${camera_lens_axis}" />
+        <limit lower="-0.5236" upper="1.5708" effort="5.0" velocity="5.24" />
     </joint>
 </robot>
